File: ESP32_SMD/ESP32_SMD.kicad_pcb (KiCad board)
At the start: 2 copper layers, 100 x 100 mm, 37 parts, among them J1 POWER, J10 INPUT_2, J11 Conn_01x15_Socket, J12 Conn_01x02_Socket, J13 Conn_01x02_Socket, J14 Conn_01x02_Socket, J15 Conn_01x02_Socket, J17 I2C, J18 Conn_01x03_Socket, J19 Conn_01x03_Socket, J2 Conn_01x02_Socket, J3 Serial Converter, J4 I2C, J5 Conn_01x02_Socket, J6 Conn_01x02_Socket, J7 Conn_01x02_Socket, J8 Conn_01x02_Socket, J9 INPUT_1, SW1 SW_Nidec_CAS-120A1, SW2 SW_DPST_x2, SW3 SW_DPST_x2, U1 ESP32-WROOM-32E, U2 R-78B1.2-2.0

Commit message: 2024/11/05
Parts:
- added D10: LED, LED_SMD:LED_0603_1608Metric_Pad1.05x0.95mm_HandSolder, F.Cu at (84.5, 61.8)
- added D11: LED, LED_SMD:LED_0603_1608Metric_Pad1.05x0.95mm_HandSolder, F.Cu at (84.6, 64.2)
- added D12: LED, LED_SMD:LED_0603_1608Metric_Pad1.05x0.95mm_HandSolder, F.Cu at (84.6, 67.0)
- added D13: LED, LED_SMD:LED_0603_1608Metric_Pad1.05x0.95mm_HandSolder, F.Cu at (84.6, 69.5)
- added D14: LED, LED_SMD:LED_0603_1608Metric_Pad1.05x0.95mm_HandSolder, F.Cu at (84.6, 72.0)
- added D15: LED, LED_SMD:LED_0603_1608Metric_Pad1.05x0.95mm_HandSolder, F.Cu at (84.6, 74.8)
- added D16: LED, LED_SMD:LED_0603_1608Metric_Pad1.05x0.95mm_HandSolder, F.Cu at (84.6, 77.0)
- added D17: LED, LED_SMD:LED_0603_1608Metric_Pad1.05x0.95mm_HandSolder, F.Cu at (84.6, 79.5)
- added D18: LED, LED_SMD:LED_0603_1608Metric_Pad1.05x0.95mm_HandSolder, F.Cu at (84.6, 82.2)
- added D19: LED, LED_SMD:LED_0603_1608Metric_Pad1.05x0.95mm_HandSolder, F.Cu at (84.6, 84.8)
- added D2: LED, LED_SMD:LED_0603_1608Metric_Pad1.05x0.95mm_HandSolder, F.Cu at (131.1, 84.8)
- added D20: LED, LED_SMD:LED_0603_1608Metric_Pad1.05x0.95mm_HandSolder, F.Cu at (84.6, 87.2)
- added D21: LED, LED_SMD:LED_0603_1608Metric_Pad1.05x0.95mm_HandSolder, F.Cu at (131.1, 69.5)
- added D22: LED, LED_SMD:LED_0603_1608Metric_Pad1.05x0.95mm_HandSolder, F.Cu at (131.1, 67.0)
- added D23: LED, LED_SMD:LED_0603_1608Metric_Pad1.05x0.95mm_HandSolder, F.Cu at (131.1, 64.5)
- added D24: LED, LED_SMD:LED_0603_1608Metric_Pad1.05x0.95mm_HandSolder, F.Cu at (131.1, 61.8)
- added D25: LED, LED_SMD:LED_0603_1608Metric_Pad1.05x0.95mm_HandSolder, F.Cu at (131.1, 59.2)
- added D26: LED, LED_SMD:LED_0603_1608Metric_Pad1.05x0.95mm_HandSolder, F.Cu at (131.1, 57.0)
- added D27: LED, LED_SMD:LED_0603_1608Metric_Pad1.05x0.95mm_HandSolder, F.Cu at (131.1, 54.2)
- added D28: LED, LED_SMD:LED_0603_1608Metric_Pad1.05x0.95mm_HandSolder, F.Cu at (131.1, 51.8)
- added D3: LED, LED_SMD:LED_0603_1608Metric_Pad1.05x0.95mm_HandSolder, F.Cu at (131.1, 82.2)
- added D4: LED, LED_SMD:LED_0603_1608Metric_Pad1.05x0.95mm_HandSolder, F.Cu at (131.1, 79.8)
- added D5: LED, LED_SMD:LED_0603_1608Metric_Pad1.05x0.95mm_HandSolder, F.Cu at (131.1, 77.0)
- added D6: LED, LED_SMD:LED_0603_1608Metric_Pad1.05x0.95mm_HandSolder, F.Cu at (131.1, 74.5)
- added D7: LED, LED_SMD:LED_0603_1608Metric_Pad1.05x0.95mm_HandSolder, F.Cu at (131.1, 72.0)
- added D8: LED, LED_SMD:LED_0603_1608Metric_Pad1.05x0.95mm_HandSolder, F.Cu at (84.5, 56.8)
- added D9: LED, LED_SMD:LED_0603_1608Metric_Pad1.05x0.95mm_HandSolder, F.Cu at (84.5, 59.2)
- added F2: MF-R050, 00a:MF-R050, F.Cu at (134.5, 98.8)
- added F3: MF-R050, 00a:MF-R050, F.Cu at (89.0, 104.0)
- added J16: Conn_01x15_Socket, Connector_PinHeader_2.54mm:PinHeader_1x15_P2.54mm_Vertical, F.Cu at (91.8, 87.3)
- added J20: Conn_01x15_Socket, Connector_PinHeader_2.54mm:PinHeader_1x15_P2.54mm_Vertical, F.Cu at (123.0, 51.8)
- added J21: Conn_01x02_Socket, Connector_JST:JST_XH_B2B-XH-A_1x02_P2.50mm_Vertical, F.Cu at (76.0, 111.2)
- added J22: Conn_01x03_Socket, Connector_JST:JST_XH_B3B-XH-A_1x03_P2.50mm_Vertical, F.Cu at (65.2, 79.8)
- added J23: Conn_01x03_Socket, Connector_JST:JST_XH_B3B-XH-A_1x03_P2.50mm_Vertical, F.Cu at (65.2, 91.2)
- added J24: Conn_01x03_Socket, Connector_JST:JST_XH_B3B-XH-A_1x03_P2.50mm_Vertical, F.Cu at (65.2, 102.8)
- added J25: POWER(3.3V), Connector_JST:JST_XH_B2B-XH-A_1x02_P2.50mm_Vertical, F.Cu at (146.2, 95.8)
- added R10: 240Ω, Resistor_SMD:R_0603_1608Metric_Pad0.98x0.95mm_HandSolder, F.Cu at (88.0, 74.8)
- added R11: 240Ω, Resistor_SMD:R_0603_1608Metric_Pad0.98x0.95mm_HandSolder, F.Cu at (88.0, 77.0)
- added R12: 240Ω, Resistor_SMD:R_0603_1608Metric_Pad0.98x0.95mm_HandSolder, F.Cu at (88.0, 79.5)
- added R13: 240Ω, Resistor_SMD:R_0603_1608Metric_Pad0.98x0.95mm_HandSolder, F.Cu at (88.0, 82.2)
- added R14: 240Ω, Resistor_SMD:R_0603_1608Metric_Pad0.98x0.95mm_HandSolder, F.Cu at (88.0, 84.8)
- added R15: 240Ω, Resistor_SMD:R_0603_1608Metric_Pad0.98x0.95mm_HandSolder, F.Cu at (88.0, 87.2)
- added R16: 240Ω, Resistor_SMD:R_0603_1608Metric_Pad0.98x0.95mm_HandSolder, F.Cu at (127.6, 84.8)
- added R17: 240Ω, Resistor_SMD:R_0603_1608Metric_Pad0.98x0.95mm_HandSolder, F.Cu at (127.6, 82.2)
- added R18: 240Ω, Resistor_SMD:R_0603_1608Metric_Pad0.98x0.95mm_HandSolder, F.Cu at (127.6, 79.8)
- added R19: 240Ω, Resistor_SMD:R_0603_1608Metric_Pad0.98x0.95mm_HandSolder, F.Cu at (127.6, 77.0)
- added R20: 240Ω, Resistor_SMD:R_0603_1608Metric_Pad0.98x0.95mm_HandSolder, F.Cu at (127.6, 74.5)
- added R21: 240Ω, Resistor_SMD:R_0603_1608Metric_Pad0.98x0.95mm_HandSolder, F.Cu at (127.6, 72.0)
- added R22: 240Ω, Resistor_SMD:R_0603_1608Metric_Pad0.98x0.95mm_HandSolder, F.Cu at (127.6, 69.5)
- added R23: 240Ω, Resistor_SMD:R_0603_1608Metric_Pad0.98x0.95mm_HandSolder, F.Cu at (127.6, 67.0)
- added R24: 240Ω, Resistor_SMD:R_0603_1608Metric_Pad0.98x0.95mm_HandSolder, F.Cu at (127.6, 64.5)
- added R25: 240Ω, Resistor_SMD:R_0603_1608Metric_Pad0.98x0.95mm_HandSolder, F.Cu at (127.6, 61.8)
- added R26: 240Ω, Resistor_SMD:R_0603_1608Metric_Pad0.98x0.95mm_HandSolder, F.Cu at (127.6, 59.2)
- added R27: 240Ω, Resistor_SMD:R_0603_1608Metric_Pad0.98x0.95mm_HandSolder, F.Cu at (127.6, 57.0)
- added R28: 240Ω, Resistor_SMD:R_0603_1608Metric_Pad0.98x0.95mm_HandSolder, F.Cu at (127.6, 54.2)
- added R29: 240Ω, Resistor_SMD:R_0603_1608Metric_Pad0.98x0.95mm_HandSolder, F.Cu at (127.6, 51.8)
- added R3: 240Ω, Resistor_SMD:R_0603_1608Metric_Pad0.98x0.95mm_HandSolder, F.Cu at (88.0, 56.8)
- added R4: 240Ω, Resistor_SMD:R_0603_1608Metric_Pad0.98x0.95mm_HandSolder, F.Cu at (88.0, 59.2)
- added R5: 240Ω, Resistor_SMD:R_0603_1608Metric_Pad0.98x0.95mm_HandSolder, F.Cu at (88.0, 61.8)
- added R6: 240Ω, Resistor_SMD:R_0603_1608Metric_Pad0.98x0.95mm_HandSolder, F.Cu at (88.0, 64.2)
- added R7: 240Ω, Resistor_SMD:R_0603_1608Metric_Pad0.98x0.95mm_HandSolder, F.Cu at (88.0, 67.0)
- added R8: 240Ω, Resistor_SMD:R_0603_1608Metric_Pad0.98x0.95mm_HandSolder, F.Cu at (88.0, 69.5)
- added R9: 240Ω, Resistor_SMD:R_0603_1608Metric_Pad0.98x0.95mm_HandSolder, F.Cu at (88.0, 72.0)
- C1, C2: footprint Capacitor_THT:C_Disc_D3.0mm_W2.0mm_P2.50mm -> Capacitor_SMD:C_0603_1608Metric_Pad1.08x0.95mm_HandSolder
- C4: value C -> 2.2μF; footprint Connector_PinHeader_2.54mm:PinHeader_1x02_P2.54mm_Vertical -> Capacitor_SMD:C_0603_1608Metric_Pad1.08x0.95mm_HandSolder
- C5: value C -> 0.33μF; footprint Connector_PinHeader_2.54mm:PinHeader_1x02_P2.54mm_Vertical -> Capacitor_SMD:C_0603_1608Metric_Pad1.08x0.95mm_HandSolder
- D1: footprint LED_THT:LED_D3.0mm_Horizontal_O6.35mm_Z10.0mm -> LED_SMD:LED_0603_1608Metric
- F1: value Polyfuse -> MF-R050; footprint 00a:RXEF005 -> 00a:MF-R050
- J1: value POWER -> POWER(5V)
- J11: value Conn_01x15_Socket -> Conn_01x02_Socket; footprint Connector_Dsub:DSUB-15_Female_Vertical_P2.77x2.84mm -> Connector_JST:JST_XH_B2B-XH-A_1x02_P2.50mm_Vertical; moved to F.Cu
- J15: value Conn_01x02_Socket -> Conn_01x03_Socket; footprint Connector_JST:JST_XH_B2B-XH-A_1x02_P2.50mm_Vertical -> Connector_JST:JST_XH_B3B-XH-A_1x03_P2.50mm_Vertical
- J3: value Serial Converter -> FT234X(Serial Converter)
- R1, R2: footprint Resistor_THT:R_Axial_DIN0207_L6.3mm_D2.5mm_P10.16mm_Horizontal -> Resistor_SMD:R_0603_1608Metric_Pad0.98x0.95mm_HandSolder
- U2: value R-78B1.2-2.0 -> NJM2845DL1-33; footprint Converter_DCDC:Converter_DCDC_RECOM_R-78B-2.0_THT -> 00a:TO-252-3_TabPin2
- moved G*** 116.1 mm to (247.2, 45.7)
- moved G*** 116.1 mm to (233.5, 46.5)
- moved J15 97.3 mm to (65.2, 67.8), turned to 90 degrees
- moved D1 74.0 mm to (135.9, 102.8), turned to 180 degrees
- moved J1 71.3 mm to (146.2, 104.5), turned to 90 degrees
- moved J3 68.2 mm to (85.8, 107.4), turned to 180 degrees
- moved R1 66.0 mm to (132.4, 102.8), turned to 0 degrees
- moved J11 61.6 mm to (75.8, 103.2), turned to 180 degrees
- moved C4 57.3 mm to (116.0, 82.6), turned to 90 degrees
- moved F1 53.4 mm to (134.5, 105.2), turned to 180 degrees
- moved C5 50.4 mm to (116.0, 86.1), turned to -90 degrees
- moved SW2 44.0 mm to (110.2, 107.8)
- moved SW1 43.2 mm to (119.8, 106.2), turned to 180 degrees
- moved C2 42.3 mm to (107.0, 100.2)
- moved SW3 41.6 mm to (99.4, 107.8)
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Connections:
- net Net-(J10-Pin_1) renamed SENSOR_VN
- net Net-(J10-Pin_2) renamed SENSOR_VP
- net Net-(J9-Pin_1) renamed IO35
- net Net-(J9-Pin_2) renamed IO34
- net Net-(SW3A-B) renamed EN
- C4 pad 1: Net-(J3-Pin_4) -> GND
- C4 pad 2: GND -> +3.3V
- C5 pad 1: Net-(U2-OUT) -> GND
- C5 pad 2: GND -> +5V
- F1 pad 1: Net-(U1-VDD) -> Net-(J1-Pin_1)
- F1 pad 2: Net-(U2-OUT) -> Net-(SW1-C)
- J11 pad 1: IO23 -> IO15
- J11 pad 2: IO17 -> IO12
- J15 pad 1: IO2 -> IO25
- J15 pad 2: IO15 -> IO33
- J17 pad 1: Net-(J17-Pin_1) -> IO21
- J17 pad 2: Net-(J17-Pin_2) -> IO22
- J18 pad 1: IO17 -> IO5
- J18 pad 2: IO12 -> IO17
- J19 pad 1: IO19 -> IO23
- J19 pad 2: IO0 -> IO19
- J2 pad 1: IO1 -> TXD0/IO1
- J2 pad 2: IO3 -> RXD0/IO3
- J3 pad 1: IO1 -> +5V_PC
- J3 pad 2: IO3 -> GND
- J3 pad 3: GND -> RXD0/IO3
- J3 pad 4: Net-(J3-Pin_4) -> TXD0/IO1
- J4 pad 1: Net-(J17-Pin_1) -> IO21
- J4 pad 2: Net-(J17-Pin_2) -> IO22
- J5 pad 1: IO13 -> IO4
- J5 pad 2: IO4 -> IO13
- R1 pad 1: Net-(D1-A) -> +3.3V
- R1 pad 2: Net-(J3-Pin_4) -> Net-(D1-A)
- R2 pad 1: Net-(U1-VDD) -> +3.3V
- SW1 pad 1: unconnected-(SW1-C-Pad1) -> Net-(SW1-C)
- SW1 pad 2: Net-(J1-Pin_1) -> +5V
- SW1 pad 3: Net-(J3-Pin_4) -> Net-(SW1-A)
- U1 pad 2: Net-(U1-VDD) -> +3.3V
- U1 pad 33: Net-(J17-Pin_2) -> IO21
- U1 pad 34: IO3 -> RXD0/IO3
- U1 pad 35: IO1 -> TXD0/IO1
- U1 pad 36: Net-(J17-Pin_1) -> IO22
- U2 pad 1: Net-(J3-Pin_4) -> +5V
- U2 pad 3: Net-(U2-OUT) -> +3.3V
Routing:
- net IO3: track 126.3 -> 0.00 mm, vias 1 -> 0
- net IO1: track 125.2 -> 0.00 mm, vias 1 -> 0
- net EN: track 129.3 -> 12.0 mm, vias 2 -> 0
- net Net-(U1-VDD): track 102.3 -> 0.00 mm
- net Net-(J3-Pin_4): track 86.4 -> 0.00 mm
- net IO32: track 130.7 -> 47.4 mm
- net +3.3V: track 0.00 -> 80.7 mm
- net IO33: track 126.4 -> 48.2 mm
- net IO26: track 116.3 -> 50.6 mm
- net IO25: track 119.2 -> 53.8 mm
- net IO0: track 159.0 -> 96.3 mm
- net IO13: track 115.4 -> 58.6 mm
- net IO27: track 110.4 -> 56.3 mm
- net IO14: track 105.9 -> 56.7 mm
- net TXD0/IO1: track 0.00 -> 39.0 mm
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- added copper zone on F.Cu, net EN
- added copper zone on F.Cu, net IO0
Other:
- board size 100 x 100 mm -> 90 x 75 mm
- copper layers 2 -> 4
- board text added: "0"
- board text added: "0.1μF"
- board text added: "1"
- board text added: "12"
- board text added: "13"
- board text added: "14"
- board text added: "15"
- board text added: "16"
- board text added: "1608 240Ω"
- board text added: "17"
- board text added: "18"
- board text added: "19"
- board text added: "2"
- board text added: "21"
- board text added: "22"
- board text added: "23"
- board text added: "25"
- board text added: "26"
- board text added: "27"
- board text added: "3"
- board text added: "3.3V"
- board text added: "32"
- board text added: "33"
- board text added: "34"
- board text added: "35"
- board text added: "36"
- board text added: "39"
- board text added: "4"
- board text added: "5"
- board text added: "5V"
- board text added: "EN"
- board text added: "GND"
- board text added: "LED OSHR1608"

Commit message: 2024/11/05/23:24
Parts:
- removed the REF** at (156.0, 54.2)
- removed the REF** at (156.0, 144.2)
- added LS1: PKM13EPYH4000-A0, 00a:PKM13EPYH4000-A0, F.Cu at (105.5, 95.5)
- added R30: 100Ω~1kΩ, Resistor_SMD:R_0603_1608Metric_Pad0.98x0.95mm_HandSolder, F.Cu at (93.0, 91.5)
- G*** (x2): moved to B.Cu
- J3: value FT234X(Serial Converter) -> FT234X
- SW2: value SW_DPST_x2 -> BOOT
- SW3: value SW_DPST_x2 -> EN
- moved G*** 142.8 mm to (113.5, 96.0), turned to 180 degrees
- moved G*** 119.5 mm to (125.0, 96.5), turned to 180 degrees
- moved REF** 33.5 mm to (66.0, 110.8)
- moved D1 12.4 mm to (129.7, 113.5), turned to 0 degrees
- moved R1 10.8 mm to (133.2, 113.5), turned to 180 degrees
- moved J1 7.36 mm to (145.0, 111.8)
- moved J25 7.36 mm to (145.0, 103.0)
- moved J3 5.70 mm to (89.1, 112.0), turned to -90 degrees
- moved C1 4.76 mm to (96.4, 105.5)
- moved C2 4.76 mm to (107.2, 105.0)
- moved R2 4.76 mm to (96.4, 103.5)
- moved SW2 4.76 mm to (110.5, 112.5)
- moved SW3 4.76 mm to (99.7, 112.5)
- moved F1 4.75 mm to (134.5, 110.0)
- moved SW1 4.24 mm to (121.6, 110.0)
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Routing:
- net TXD0/IO1: track 39.0 -> 114.2 mm
- net RXD0/IO3: track 35.7 -> 104.0 mm
- net +3.3V: track 80.7 -> 143.5 mm
- net +5V: track 0.00 -> 51.9 mm
- net EN: track 12.0 -> 62.2 mm, vias 0 -> 1
- net Net-(SW1-A): track 0.00 -> 34.9 mm
- net Net-(LS1-Pad2): track 0.00 -> 10.7 mm
- net Net-(SW1-C): track 0.00 -> 9.12 mm
- net Net-(J1-Pin_1): track 0.00 -> 7.40 mm
- net Net-(J25-Pin_1): track 0.00 -> 6.88 mm
- net IO13: track 58.6 -> 63.5 mm
- net +5V_PC: track 0.00 -> 4.23 mm
- net IO32: track 47.4 -> 50.9 mm
- net IO33: track 48.2 -> 49.4 mm
- net IO26: track 50.6 -> 51.8 mm
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Other:
- board size 90 x 75 mm -> 90 x 66 mm
- board text added: "+"
- board text added: "-"
- board text added: "21(SDA)"
- board text added: "22(SCL)"
- board text added: "240Ω"
- board text added: "ESP32_SMD_v2.0.0"
- board text added: "INPUT_ONLY"
- board text added: "PC"
- board text added: "POWER(3.3V)"
- board text added: "RxD"
- board text added: "TxD"
- board text added: "VBAT"
- board text added: "https://github.com/syamei0/kicad"
- board text added: "⇔"
- board text added: "右下のスイッチでPC給電と電源基盤給電 を変更できます。 I2Cは右上の破線部分に２つあります。 bootモードのやり方 ・BOOTボタンを押す(押しっぱなし) ・ENボタンを押す ・ENボタンを離す ・BOOTボタンを離す 2024/11/05 Yamamoto Maku"
- board text removed: "0.1μF"
- board text removed: "ESP32_SMD_v1.1.0"

Commit message: 2024/11/18
Parts:
- removed F3: MF-R050, 00a:MF-R050
- removed the REF** at (66.0, 110.8)
- removed the REF** at (66.0, 54.2)
- added REF**: MountingHole_3.2mm_M3, MountingHole:MountingHole_3.2mm_M3, F.Cu at (154.0, 48.5)
- added REF**: MountingHole_3.2mm_M3, MountingHole:MountingHole_3.2mm_M3, F.Cu at (63.2, 48.5)
- added REF**: MountingHole_3.2mm_M3, MountingHole:MountingHole_3.2mm_M3, F.Cu at (154.0, 114.8)
- added REF**: MountingHole_3.2mm_M3, MountingHole:MountingHole_3.2mm_M3, F.Cu at (63.2, 114.8)
- R10, R11, R12, R13, R14, R15, R16, R17, R18, R19, R20, R21, R22, R23, R24, R25, R26, R27, R28, R29, R3, R4, R5, R6, R7, R8, R9: value 240Ω -> 1kΩ
- moved G*** 29.5 mm to (95.5, 98.0)
- moved G*** 29.5 mm to (84.0, 97.5)
- moved F1 19.5 mm to (118.8, 98.5), turned to 90 degrees
Connections:
- F1 pad 1: Net-(J1-Pin_1) -> Net-(SW1-B)
- F1 pad 2: Net-(SW1-C) -> +5V
- SW1 pad 1: Net-(SW1-C) -> Net-(J1-Pin_1)
- SW1 pad 2: +5V -> Net-(SW1-B)
- SW1 pad 3: Net-(SW1-A) -> +5V_PC
Routing:
- net Net-(SW1-A): track 34.9 -> 0.00 mm
- net +5V: track 51.9 -> 21.3 mm
- net +5V_PC: track 4.23 -> 28.4 mm
- net Net-(J1-Pin_1): track 7.40 -> 24.1 mm
- net Net-(SW1-C): track 9.12 -> 0.00 mm
- net Net-(SW1-B): track 0.00 -> 7.82 mm
Other:
- board size 90 x 66 mm -> 96.8 x 72.2 mm
- board text added: "1608 1kΩ"
- board text added: "1kΩ"
- board text added: "ESP32_SMD_v2.1.0"
- board text removed: "1608 240Ω"
- board text removed: "240Ω"
- board text removed: "ESP32_SMD_v2.0.0"
