File: ESP32_SMD/ESP32_SMD.kicad_sch (KiCad schematic)
At the start: 30 parts, among them J1 POWER, J10 INPUT_2, J11 Conn_01x15_Socket, J12 Conn_01x02_Socket, J13 Conn_01x02_Socket, J14 Conn_01x02_Socket, J15 Conn_01x02_Socket, J17 I2C, J18 Conn_01x03_Socket, J19 Conn_01x03_Socket, J2 Conn_01x02_Socket, J3 Serial Converter, J4 I2C, J5 Conn_01x02_Socket, J6 Conn_01x02_Socket, J7 Conn_01x02_Socket, J8 Conn_01x02_Socket, J9 INPUT_1, SW1 SW_Nidec_CAS-120A1, SW2 SW_DPST_x2, SW3 SW_DPST_x2, U1 ESP32-WROOM-32E, U2 R-78B1.2-2.0

Commit message: 2024/10/15
Parts:
- added R2: 10kΩ, Resistor_THT:R_Axial_DIN0207_L6.3mm_D2.5mm_P10.16mm_Horizontal, symbol Device:R
- R1: value R -> 240Ω
Connections:
- net IO1: now also J3.1 (Pin_1); no longer J3.2 (Pin_2)
- net IO3: now also J3.2 (Pin_2); no longer J3.1 (Pin_1)
- net at C1.1, SW3.2 (B), U1.3 (EN): now also R2.2
- net at F1.1, U1.2 (VDD): now also R2.1
Changed lines of the file:
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@@
 	)
 	(junction
+		(at 83.82 160.02)
+		(diameter 0)
+		(color 0 0 0 0)
+	)
+	(junction
 		(at 35.56 167.64)
 		(diameter 0)
@@
 	)
 	(junction
+		(at 91.44 166.37)
+		(diameter 0)
+		(color 0 0 0 0)
+	)
+	(junction
 		(at 167.64 66.04)
 		(diameter 0)
@@
 	(wire
 		(pts
+			(xy 170.18 189.23) (xy 171.45 189.23)
+		)
+		(stroke
+			(width 0)
+			(type default)
+		)
+	)
+	(wire
+		(pts
 			(xy 166.37 105.41) (xy 199.39 105.41)
 		)
@@
 	(wire
 		(pts
+			(xy 91.44 166.37) (xy 91.44 177.8)
+		)
+		(stroke
+			(width 0)
+			(type default)
+		)
+	)
+	(wire
+		(pts
+			(xy 83.82 160.02) (xy 71.12 160.02)
+		)
+		(stroke
+			(width 0)
+			(type default)
+		)
+	)
+	(wire
+		(pts
 			(xy 175.26 123.19) (xy 175.26 88.9)
 		)
@@
 	(wire
 		(pts
-			(xy 167.64 189.23) (xy 171.45 189.23)
+			(xy 153.67 63.5) (xy 153.67 43.18)
 		)
 		(stroke
@@
 	(wire
 		(pts
-			(xy 153.67 63.5) (xy 153.67 43.18)
+			(xy 166.37 76.2) (xy 166.37 105.41)
 		)
 		(stroke
@@
 	(wire
 		(pts
-			(xy 166.37 76.2) (xy 166.37 105.41)
+			(xy 146.05 76.2) (xy 166.37 76.2)
 		)
 		(stroke
@@
 	(wire
 		(pts
-			(xy 146.05 76.2) (xy 166.37 76.2)
+			(xy 167.64 66.04) (xy 167.64 186.69)
 		)
 		(stroke
@@
 	(wire
 		(pts
-			(xy 167.64 66.04) (xy 167.64 189.23)
+			(xy 165.1 110.49) (xy 199.39 110.49)
 		)
 		(stroke
@@
 	(wire
 		(pts
-			(xy 165.1 110.49) (xy 199.39 110.49)
+			(xy 92.71 177.8) (xy 92.71 190.5)
 		)
 		(stroke
@@
 	(wire
 		(pts
-			(xy 92.71 177.8) (xy 92.71 190.5)
+			(xy 167.64 186.69) (xy 171.45 186.69)
 		)
 		(stroke
@@
 	(wire
 		(pts
-			(xy 91.44 63.5) (xy 91.44 177.8)
+			(xy 91.44 63.5) (xy 91.44 166.37)
 		)
 		(stroke
@@
 	(wire
 		(pts
-			(xy 87.63 160.02) (xy 71.12 160.02)
+			(xy 87.63 160.02) (xy 83.82 160.02)
 		)
 		(stroke
@@
 	(wire
 		(pts
-			(xy 170.18 186.69) (xy 171.45 186.69)
-		)
-		(stroke
-			(width 0)
-			(type default)
-		)
-	)
-	(wire
-		(pts
 			(xy 148.59 88.9) (xy 148.59 92.71)
 		)
@@
 	(wire
 		(pts
+			(xy 83.82 160.02) (xy 83.82 166.37)
+		)
+		(stroke
+			(width 0)
+			(type default)
+		)
+	)
+	(wire
+		(pts
 			(xy 175.26 76.2) (xy 175.26 63.5)
 		)
@@
 	(wire
 		(pts
-			(xy 170.18 68.58) (xy 170.18 186.69)
+			(xy 170.18 68.58) (xy 170.18 189.23)
 		)
 		(stroke
@@
 			)
 		)
-		(property "Value" "R"
+		(property "Value" "240Ω"
 			(at 20.32 175.2599 0)
 			(effects
@@
 					(unit 1)
 				)
+			)
+		)
+	)
+	(symbol
+		(lib_id "Device:R")
+		(at 87.63 166.37 90)
+		(unit 1)
+		(exclude_from_sim no)
+		(in_bom yes)
+		(on_board yes)
+		(dnp no)
+		(fields_autoplaced yes)
+		(property "Reference" "R2"
+			(at 87.63 160.02 90)
+			(effects
+				(font
+					(size 1.27 1.27)
+				)
+			)
+		)
+		(property "Value" "10kΩ"
+			(at 87.63 162.56 90)
+			(effects
+				(font
+					(size 1.27 1.27)
+				)
+			)
+		)
+		(property "Footprint" "Resistor_THT:R_Axial_DIN0207_L6.3mm_D2.5mm_P10.16mm_Horizontal"
+			(at 87.63 168.148 90)
+			(effects
+				(font
+					(size 1.27 1.27)
+				)
+				(hide yes)
+			)
+		)
+		(property "Datasheet" "~"
+			(at 87.63 166.37 0)
+			(effects
+				(font
+					(size 1.27 1.27)
+				)
+				(hide yes)
+			)
+		)
+		(property "Description" "Resistor"
+			(at 87.63 166.37 0)
+			(effects
+				(font
+					(size 1.27 1.27)
+				)
+				(hide yes)
+			)
+		)
+		(pin "1"
+		)
+		(pin "2"
+		)
+		(instances
+			(project ""
+				(path "/16d7c20d-89b8-473d-a0a1-bcb2e2ab28b6"
+					(reference "R2")
+					(unit 1)
+				)

Commit message: 2024/11/05
Parts:
- removed J11: Conn_01x15_Socket, Connector_Dsub:DSUB-15_Female_Vertical_P2.77x2.84mm, symbol Connector:Conn_01x15_Socket
- removed J15: Conn_01x02_Socket, Connector_JST:JST_XH_B2B-XH-A_1x02_P2.50mm_Vertical, symbol Connector:Conn_01x02_Socket
- added D10, D11, D12, D13, D14, D15, D16, D17, D18, D19, D2, D20, D21, D22, D23, D24, D25, D26, D27, D28, D3, D4, D5, D6, D7, D8, D9: LED, LED_SMD:LED_0603_1608Metric_Pad1.05x0.95mm_HandSolder, symbol Device:LED
- added F2, F3: MF-R050, 00a:MF-R050, symbol Device:Polyfuse
- added J11, J21: Conn_01x02_Socket, Connector_JST:JST_XH_B2B-XH-A_1x02_P2.50mm_Vertical, symbol Connector:Conn_01x02_Socket
- added J15, J22, J23, J24: Conn_01x03_Socket, Connector_JST:JST_XH_B3B-XH-A_1x03_P2.50mm_Vertical, symbol Connector:Conn_01x03_Socket
- added J16, J20: Conn_01x15_Socket, Connector_PinHeader_2.54mm:PinHeader_1x15_P2.54mm_Vertical, symbol Connector:Conn_01x15_Socket
- added J25: POWER(3.3V), Connector_JST:JST_XH_B2B-XH-A_1x02_P2.50mm_Vertical, symbol Connector:Conn_01x02_Socket
- added R10, R11, R12, R13, R14, R15, R16, R17, R18, R19, R20, R21, R22, R23, R24, R25, R26, R27, R28, R29, R3, R4, R5, R6, R7, R8, R9: 240Ω, Resistor_SMD:R_0603_1608Metric_Pad0.98x0.95mm_HandSolder, symbol Device:R
- C1, C2: footprint Capacitor_THT:C_Disc_D3.0mm_W2.0mm_P2.50mm -> Capacitor_SMD:C_0603_1608Metric_Pad1.08x0.95mm_HandSolder
- C4: value C -> 2.2μF; footprint Connector_PinHeader_2.54mm:PinHeader_1x02_P2.54mm_Vertical -> Capacitor_SMD:C_0603_1608Metric_Pad1.08x0.95mm_HandSolder
- C5: value C -> 0.33μF; footprint Connector_PinHeader_2.54mm:PinHeader_1x02_P2.54mm_Vertical -> Capacitor_SMD:C_0603_1608Metric_Pad1.08x0.95mm_HandSolder
- D1: footprint LED_THT:LED_D3.0mm_Horizontal_O6.35mm_Z10.0mm -> LED_SMD:LED_0603_1608Metric
- F1: value Polyfuse -> MF-R050; footprint 00a:RXEF005 -> 00a:MF-R050
- J1: value POWER -> POWER(5V)
- J3: value Serial Converter -> FT234X(Serial Converter)
- R1, R2: footprint Resistor_THT:R_Axial_DIN0207_L6.3mm_D2.5mm_P10.16mm_Horizontal -> Resistor_SMD:R_0603_1608Metric_Pad0.98x0.95mm_HandSolder
- U2: value R-78B1.2-2.0 -> NJM2845DL1-33; footprint Converter_DCDC:Converter_DCDC_RECOM_R-78B-2.0_THT -> 00a:TO-252-3_TabPin2
Connections:
- net GND: now also C4.1, C5.1, J3.2 (GND), D10.1 (K), D11.1 (K), D12.1 (K), D13.1 (K), D14.1 (K), D15.1 (K), D16.1 (K), D17.1 (K), D18.1 (K), D19.1 (K), D2.1 (K), D20.1 (K), D21.1 (K), D22.1 (K), D23.1 (K), D24.1 (K), D25.1 (K), D26.1 (K), D27.1 (K), D28.1 (K), D3.1 (K), D4.1 (K), D5.1 (K), D6.1 (K), D7.1 (K), D8.1 (K), D9.1 (K), J16.15 (Pin_15), J25.2 (Pin_2); no longer C4.2, C5.2, J3.3 (Pin_3)
- net IO0: now also J20.12 (Pin_12), J21.1 (Pin_1), J24.1 (Pin_1), R18.2; no longer J19.2 (Pin_2)
- net IO12: now also J11.2 (Pin_2), J16.2 (Pin_2), J23.1 (Pin_1), R14.2; no longer J18.2 (Pin_2)
- net IO13: now also J5.2 (Pin_2), J16.1 (Pin_1), J23.3 (Pin_3), R15.2; no longer J5.1 (Pin_1)
- net IO14: now also J16.3 (Pin_3), J22.1 (Pin_1), R13.2
- net IO15: now also J11.1 (Pin_1), J20.14 (Pin_14), J24.3 (Pin_3), R16.2
- net IO16: now also J20.10 (Pin_10), R20.2
- net IO17: now also J18.2 (Pin_2), J20.9 (Pin_9), R21.2; no longer J18.1 (Pin_1)
- net IO18: now also J20.7 (Pin_7), R23.2
- net IO19: now also J19.2 (Pin_2), J20.6 (Pin_6), R24.2; no longer J19.1 (Pin_1)
- net IO2: now also J20.13 (Pin_13), J21.2 (Pin_2), J24.2 (Pin_2), R17.2
- net IO23: now also J19.1 (Pin_1), J20.1 (Pin_1), R29.2
- net IO25: now also J15.1 (Pin_1), J16.6 (Pin_6), R10.2
- net IO26: now also J16.5 (Pin_5), J22.3 (Pin_3), R11.2
- net IO27: now also J16.4 (Pin_4), J22.2 (Pin_2), R12.2
- net IO32: now also J15.3 (Pin_3), J16.8 (Pin_8), R8.2
- net IO33: now also J15.2 (Pin_2), J16.7 (Pin_7), R9.2
- net IO4: now also J5.1 (Pin_1), J20.11 (Pin_11), J23.2 (Pin_2), R19.2; no longer J5.2 (Pin_2)
- net IO5: now also J18.1 (Pin_1), J20.8 (Pin_8), R22.2
- net EN: now reaches C1.1, R2.2, SW3.2 (B), U1.3 (EN)
- net EN: now also J16.13 (Pin_13), R3.2
- net IO35: now reaches J9.1 (Pin_1), U1.7 (IO35)
- net IO35: now also J16.9 (Pin_9), R7.2
- net IO34: now reaches J9.2 (Pin_2), U1.6 (IO34)
- net IO34: now also J16.10 (Pin_10), R6.2
- net IO21: now reaches J17.1 (Pin_1), J4.1 (Pin_1)
- net IO21: now also U1.33 (IO21), J20.5 (Pin_5), R25.2; no longer U1.36 (IO22)
- net IO22: now reaches J17.2 (Pin_2), J4.2 (Pin_2)
- net IO22: now also U1.36 (IO22), J20.2 (Pin_2), R28.2; no longer U1.33 (IO21)
- net SENSOR_VN: now reaches J10.1 (Pin_1), U1.5 (SENSOR_VN)
- net SENSOR_VN: now also J16.11 (Pin_11), R5.2
- net SENSOR_VP: now reaches J10.2 (Pin_2), U1.4 (SENSOR_VP)
- net SENSOR_VP: now also J16.12 (Pin_12), R4.2
- net at D1.2 (A): now also R1.2; no longer R1.1
- net at J1.1 (Pin_1): now also F1.1; no longer SW1.2 (B)
- net +3.3V: now reaches R2.1, U1.2 (VDD)
- net +3.3V: now also C4.2, R1.1, U2.3 (OUT), F2.2, J16.14 (Pin_14); no longer F1.1
- net at SW1.1 (C): now also F1.2
- net IO1 renamed TXD0/IO1
- net TXD0/IO1: now also J3.4 (RxD), J20.3 (Pin_3), R27.2; no longer J3.1 (Pin_1)
- net IO3 renamed RXD0/IO3
- net RXD0/IO3: now also J3.3 (TxD), J20.4 (Pin_4), R26.2; no longer J3.2 (Pin_2)
- new net: D28.2 (A), R29.1
- new net: D7.2 (A), R21.1
- new net: D6.2 (A), R20.1
- new net: D23.2 (A), R24.1
- new net: D2.2 (A), R16.1
- new net: D8.2 (A), R3.1
- new net: D20.2 (A), R15.1
- new net: D13.2 (A), R8.1
- new net: D18.2 (A), R13.1
- new net: D25.2 (A), R26.1
- new net: D16.2 (A), R11.1
- new net: D27.2 (A), R28.1
- new net: D4.2 (A), R18.1
- new net: D15.2 (A), R10.1
- new net: F3.2, SW1.3 (A)
- new net: D21.2 (A), R22.1
- new net: F2.1, J25.1 (Pin_1)
- new net: D22.2 (A), R23.1
- new net: D24.2 (A), R25.1
- new net: D26.2 (A), R27.1
- new net: D17.2 (A), R12.1
- new net: D12.2 (A), R7.1
- new net: D10.2 (A), R5.1
- new net: D11.2 (A), R6.1
- new net: D9.2 (A), R4.1
- new net: D3.2 (A), R17.1
- new net: D14.2 (A), R9.1
- new net: D19.2 (A), R14.1
- new net: D5.2 (A), R19.1
- new net +5V: C5.2, J20.15 (Pin_15), SW1.2 (B), U2.1 (IN)
- new net +5V_PC: F3.1, J3.1 (5V)
- no-connect marks 1 -> 0
Other:
- note added: "PWM"
- note removed: "Motor"
- moved on the sheet: C1, C2, C4, C5, D1, F1, J1, J10, J12, J13, J14, J17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

Commit message: 2024/11/05/23:24
Parts:
- added LS1: PKM13EPYH4000-A0, 00a:PKM13EPYH4000-A0, symbol Device:Speaker
- added R30: 100Ω~1kΩ, Resistor_SMD:R_0603_1608Metric_Pad0.98x0.95mm_HandSolder, symbol Device:R
- J3: value FT234X(Serial Converter) -> FT234X
- SW2: value SW_DPST_x2 -> BOOT
- SW3: value SW_DPST_x2 -> EN
Connections:
- net GND: now also LS1.1
- net IO13: now also R30.2
- new net: LS1.2, R30.1
Changed lines of the file:
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@@
 	(wire
 		(pts
+			(xy 110.49 140.97) (xy 127 140.97)
+		)
+		(stroke
+			(width 0)
+			(type default)
+		)
+	)
+	(wire
+		(pts
 			(xy 151.13 87.63) (xy 151.13 92.71)
 		)
@@
 	(wire
 		(pts
+			(xy 134.62 140.97) (xy 156.21 140.97)
+		)
+		(stroke
+			(width 0)
+			(type default)
+		)
+	)
+	(wire
+		(pts
 			(xy 88.9 90.17) (xy 88.9 121.92)
 		)
@@
 		)
 	)
+	(global_label "IO13"
+		(shape bidirectional)
+		(at 156.21 140.97 0)
+		(fields_autoplaced yes)
+		(effects
+			(font
+				(size 1.27 1.27)
+			)
+			(justify left)
+		)
+		(property "Intersheetrefs" "${INTERSHEET_REFS}"
+			(at 164.6608 140.97 0)
+			(effects
+				(font
+					(size 1.27 1.27)
+				)
+				(justify left)
+				(hide yes)
+			)
+		)
+	)
 	(global_label "IO33"
 		(shape bidirectional)
@@
 			)
 		)
-		(property "Value" "FT234X(Serial Converter)"
+		(property "Value" "FT234X"
 			(at 238.76 127.762 0)
 			(effects
@@
 			)
 		)
-		(property "Value" "SW_DPST_x2"
+		(property "Value" "EN"
 			(at 123.19 184.15 0)
 			(effects
@@
 	)
 	(symbol
+		(lib_id "power:GND")
+		(at 110.49 143.51 90)
+		(unit 1)
+		(exclude_from_sim no)
+		(in_bom yes)
+		(on_board yes)
+		(dnp no)
+		(fields_autoplaced yes)
+		(property "Reference" "#PWR022"
+			(at 116.84 143.51 0)
+			(effects
+				(font
+					(size 1.27 1.27)
+				)
+				(hide yes)
+			)
+		)
+		(property "Value" "GND"
+			(at 114.3 143.5099 90)
+			(effects
+				(font
+					(size 1.27 1.27)
+				)
+				(justify right)
+			)
+		)
+		(property "Footprint" ""
+			(at 110.49 143.51 0)
+			(effects
+				(font
+					(size 1.27 1.27)
+				)
+				(hide yes)
+			)
+		)
+		(property "Datasheet" ""
+			(at 110.49 143.51 0)
+			(effects
+				(font
+					(size 1.27 1.27)
+				)
+				(hide yes)
+			)
+		)
+		(property "Description" "Power symbol creates a global label with name \"GND\" , ground"
+			(at 110.49 143.51 0)
+			(effects
+				(font
+					(size 1.27 1.27)
+				)
+				(hide yes)
+			)
+		)
+		(pin "1"
+		)
+		(instances
+			(project ""
+				(path "/16d7c20d-89b8-473d-a0a1-bcb2e2ab28b6"
+					(reference "#PWR022")
+					(unit 1)
+				)
+			)
+		)
+	)
+	(symbol
 		(lib_id "Connector:Conn_01x02_Socket")
 		(at 72.39 87.63 180)
@@
 	(symbol
 		(lib_id "Device:R")
+		(at 130.81 140.97 90)
+		(unit 1)
+		(exclude_from_sim no)
+		(in_bom yes)
+		(on_board yes)
+		(dnp no)
+		(fields_autoplaced yes)
+		(property "Reference" "R30"
+			(at 130.81 134.62 90)
+			(effects
+				(font
+					(size 1.27 1.27)
+				)
+			)
+		)
+		(property "Value" "100Ω~1kΩ"
+			(at 130.81 137.16 90)
+			(effects
+				(font
+					(size 1.27 1.27)
+				)
+			)
+		)
+		(property "Footprint" "Resistor_SMD:R_0603_1608Metric_Pad0.98x0.95mm_HandSolder"
+			(at 130.81 142.748 90)
+			(effects
+				(font
+					(size 1.27 1.27)
+				)
+				(hide yes)
+			)
+		)
+		(property "Datasheet" "~"
+			(at 130.81 140.97 0)
+			(effects
+				(font
+					(size 1.27 1.27)
+				)
+				(hide yes)
+			)
+		)
+		(property "Description" "Resistor"
+			(at 130.81 140.97 0)
+			(effects
+				(font
+					(size 1.27 1.27)
+				)
+				(hide yes)
+			)
+		)
+		(pin "2"
+		)
+		(pin "1"
+		)
+		(instances
+			(project "ESP32_SMD"
+				(path "/16d7c20d-89b8-473d-a0a1-bcb2e2ab28b6"
+					(reference "R30")
+					(unit 1)
+				)
+			)
+		)
+	)
+	(symbol
+		(lib_id "Device:R")
 		(at 232.41 49.53 90)
 		(unit 1)
@@
 			)
 		)
-		(property "Value" "SW_DPST_x2"
+		(property "Value" "BOOT"
 			(at 158.75 185.42 0)
 			(effects
@@
 					(unit 1)
 				)
+			)
+		)
+	)
+	(symbol
+		(lib_id "Device:Speaker")
+		(at 105.41 143.51 180)
+		(unit 1)
+		(exclude_from_sim no)
+		(in_bom yes)
+		(on_board yes)
+		(dnp no)
+		(fields_autoplaced yes)
+		(property "Reference" "LS1"
+			(at 104.902 132.08 0)
+			(effects
+				(font
+					(size 1.27 1.27)
+				)
+			)
+		)
+		(property "Value" "PKM13EPYH4000-A0"
+			(at 104.902 134.62 0)
+			(effects
+				(font
+					(size 1.27 1.27)
+				)
+			)
+		)
+		(property "Footprint" "00a:PKM13EPYH4000-A0"
+			(at 105.41 138.43 0)
+			(effects
+				(font
+					(size 1.27 1.27)
+				)
+				(hide yes)
+			)
+		)
+		(property "Datasheet" "~"
+			(at 105.664 142.24 0)
+			(effects
+				(font
+					(size 1.27 1.27)
+				)
+				(hide yes)
+			)
+		)
+		(property "Description" "Speaker"
+			(at 105.41 143.51 0)
+			(effects
+				(font
+					(size 1.27 1.27)
+				)
+				(hide yes)
+			)
+		)
+		(pin "2"
+		)
+		(pin "1"
+		)
+		(instances
+			(project ""
+				(path "/16d7c20d-89b8-473d-a0a1-bcb2e2ab28b6"
+					(reference "LS1")
+					(unit 1)
+				)

Commit message: 2024/11/18
Parts:
- removed F3: MF-R050, 00a:MF-R050, symbol Device:Polyfuse
- R10, R11, R12, R13, R14, R15, R16, R17, R18, R19, R20, R21, R22, R23, R24, R25, R26, R27, R28, R29, R3, R4, R5, R6, R7, R8, R9: value 240Ω -> 1kΩ
Connections:
- net +5V: now also F1.2; no longer SW1.2 (B)
- net +5V_PC: now also SW1.3 (A)
- net at J1.1 (Pin_1): now also SW1.1 (C); no longer F1.1
- new net: F1.1, SW1.2 (B)
Other:
- moved on the sheet: F1, SW1
Changed lines of the file:
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@@
 	(wire
 		(pts
+			(xy 60.96 187.96) (xy 63.5 187.96)
+		)
+		(stroke
+			(width 0)
+			(type default)
+		)
+	)
+	(wire
+		(pts
 			(xy 148.59 59.69) (xy 170.18 59.69)
 		)
@@
 	(wire
 		(pts
-			(xy 27.94 190.5) (xy 40.64 190.5)
+			(xy 27.94 190.5) (xy 50.8 190.5)
 		)
 		(stroke
@@
 	(wire
 		(pts
+			(xy 71.12 187.96) (xy 73.66 187.96)
+		)
+		(stroke
+			(width 0)
+			(type default)
+		)
+	)
+	(wire
+		(pts
 			(xy 250.19 68.58) (xy 250.19 73.66)
 		)
@@
 	(wire
 		(pts
-			(xy 48.26 190.5) (xy 55.88 190.5)
-		)
-		(stroke
-			(width 0)
-			(type default)
-		)
-	)
-	(wire
-		(pts
 			(xy 97.79 72.39) (xy 118.11 72.39)
 		)
@@
 	(wire
 		(pts
-			(xy 48.26 185.42) (xy 55.88 185.42)
-		)
-		(stroke
-			(width 0)
-			(type default)
-		)
-	)
-	(wire
-		(pts
-			(xy 30.48 185.42) (xy 40.64 185.42)
+			(xy 30.48 185.42) (xy 50.8 185.42)
 		)
 		(stroke
@@
 			)
 		)
-		(property "Value" "240Ω"
+		(property "Value" "1kΩ"
 			(at 273.05 55.118 90)
 			(effects
@@
 			)
 		)
-		(property "Value" "240Ω"
+		(property "Value" "1kΩ"
 			(at 273.05 76.708 90)
 			(effects
@@
 			)
 		)
-		(property "Value" "240Ω"
+		(property "Value" "1kΩ"
 			(at 273.05 20.828 90)
 			(effects
@@
 	(symbol
 		(lib_id "power:+5V")
-		(at 66.04 187.96 270)
+		(at 73.66 187.96 270)
 		(unit 1)
 		(exclude_from_sim no)
@@
 		(fields_autoplaced yes)
 		(property "Reference" "#PWR05"
-			(at 62.23 187.96 0)
+			(at 69.85 187.96 0)
 			(effects
 				(font
@@
 		)
 		(property "Value" "+5V"
-			(at 69.85 187.9599 90)
+			(at 77.47 187.9599 90)
 			(effects
 				(font
@@
 		)
 		(property "Footprint" ""
-			(at 66.04 187.96 0)
+			(at 73.66 187.96 0)
 			(effects
 				(font
@@
 		)
 		(property "Datasheet" ""
-			(at 66.04 187.96 0)
+			(at 73.66 187.96 0)
 			(effects
 				(font
@@
 		)
 		(property "Description" "Power symbol creates a global label with name \"+5V\""
-			(at 66.04 187.96 0)
+			(at 73.66 187.96 0)
 			(effects
 				(font
@@
 			)
 		)
-		(property "Value" "240Ω"
+		(property "Value" "1kΩ"
 			(at 232.41 53.848 90)
 			(effects
@@
 			)
 		)
-		(property "Value" "240Ω"
+		(property "Value" "1kΩ"
 			(at 232.41 88.138 90)
 			(effects
@@
 			)
 		)
-		(property "Value" "240Ω"
+		(property "Value" "1kΩ"
 			(at 232.41 22.098 90)
 			(effects
@@
 			)
 		)
-		(property "Value" "240Ω"
+		(property "Value" "1kΩ"
 			(at 273.05 105.918 90)
 			(effects
@@
 			)
 		)
-		(property "Value" "240Ω"
+		(property "Value" "1kΩ"
 			(at 273.05 33.528 90)
 			(effects
@@
 	)
 	(symbol
-		(lib_id "Device:Polyfuse")
-		(at 44.45 190.5 90)
-		(unit 1)
-		(exclude_from_sim no)
-		(in_bom yes)
-		(on_board yes)
-		(dnp no)
-		(property "Reference" "F3"
-			(at 44.45 192.786 90)
-			(effects
-				(font
-					(size 1.27 1.27)
-				)
-			)
-		)
-		(property "Value" "MF-R050"
-			(at 44.45 195.072 90)
-			(effects
-				(font
-					(size 1.27 1.27)
-				)
-			)
-		)
-		(property "Footprint" "00a:MF-R050"
-			(at 50.546 190.246 0)
-			(effects
-				(font
-					(size 1.27 1.27)
-				)
-				(justify left)
-				(hide yes)
-			)
-		)
-		(property "Datasheet" "~"
-			(at 44.45 190.5 0)
-			(effects
-				(font
-					(size 1.27 1.27)
-				)
-				(hide yes)
-			)
-		)
-		(property "Description" "Resettable fuse, polymeric positive temperature coefficient"
-			(at 44.45 190.5 0)
-			(effects
-				(font
-					(size 1.27 1.27)
-				)
-				(hide yes)
-			)
-		)
-		(pin "1"
-		)
-		(pin "2"
-		)
-		(instances
-			(project "ESP32_SMD"
-				(path "/16d7c20d-89b8-473d-a0a1-bcb2e2ab28b6"
-					(reference "F3")
-					(unit 1)
-				)
-			)
-		)
-	)
-	(symbol
 		(lib_id "power:GND")
 		(at 35.56 171.45 180)
@@
 			)
 		)
-		(property "Value" "240Ω"
+		(property "Value" "1kΩ"
 			(at 273.05 69.088 90)
 			(effects
@@
 			)
 		)
-		(property "Value" "240Ω"
+		(property "Value" "1kΩ"
 			(at 273.05 84.328 90)
 			(effects
@@
 			)
 		)
-		(property "Value" "240Ω"
+		(property "Value" "1kΩ"
 			(at 232.41 75.438 90)
 			(effects
@@
 			)
 		)
-		(property "Value" "240Ω"
+		(property "Value" "1kΩ"
 			(at 273.05 91.948 90)
 			(effects
@@
 			)
 		)
-		(property "Value" "240Ω"
+		(property "Value" "1kΩ"
 			(at 273.05 99.568 90)
 			(effects
@@
 			)
 		)
-		(property "Value" "240Ω"
+		(property "Value" "1kΩ"
 			(at 273.05 61.468 90)
 			(effects
@@
 			)
 		)
-		(property "Value" "240Ω"
+		(property "Value" "1kΩ"
 			(at 232.41 47.498 90)
 			(effects
@@
 			)
 		)
-		(property "Value" "240Ω"
+		(property "Value" "1kΩ"
 			(at 232.41 34.798 90)
 			(effects
@@
 			)
 		)
-		(property "Value" "240Ω"
+		(property "Value" "1kΩ"
 			(at 232.41 41.148 90)
 			(effects
@@
 			)
 		)
-		(property "Value" "240Ω"
+		(property "Value" "1kΩ"
 			(at 273.05 113.538 90)
 			(effects
@@
 			)
 		)
-		(property "Value" "240Ω"
+		(property "Value" "1kΩ"
 			(at 232.41 28.194 90)
 			(effects
@@
 			)
 		)
-		(property "Value" "240Ω"
+		(property "Value" "1kΩ"
 			(at 273.05 27.178 90)
 			(effects
@@
 			)
 		)
-		(property "Value" "240Ω"
+		(property "Value" "1kΩ"
 			(at 232.41 60.198 90)
 			(effects
@@
 			)
 		)
-		(property "Value" "240Ω"
+		(property "Value" "1kΩ"
 			(at 232.41 94.488 90)
 			(effects
@@
 			)
 		)
-		(property "Value" "240Ω"
+		(property "Value" "1kΩ"
 			(at 273.05 48.768 90)
 			(effects
@@
 			)
 		)
-		(property "Value" "240Ω"
+		(property "Value" "1kΩ"
 			(at 273.05 41.148 90)
 			(effects
@@
 			)
 		)
-		(property "Value" "240Ω"
+		(property "Value" "1kΩ"
 			(at 232.41 67.818 90)
 			(effects
@@
 	(symbol
 		(lib_id "Switch:SW_Nidec_CAS-120A1")
-		(at 60.96 187.96 180)
+		(at 55.88 187.96 180)
 		(unit 1)
 		(exclude_from_sim no)
@@
 		(dnp no)
 		(property "Reference" "SW1"
-			(at 62.992 182.626 0)
+			(at 57.912 182.626 0)
 			(effects
 				(font
@@
 		)
 		(property "Value" "SW_Nidec_CAS-120A1"
-			(at 71.374 180.34 0)
+			(at 66.294 180.34 0)
 			(effects
 				(font
@@
 		)
 		(property "Footprint" "TerminalBlock:TerminalBlock_Xinya_XY308-2.54-3P_1x03_P2.54mm_Horizontal"
-			(at 60.96 177.8 0)
+			(at 55.88 177.8 0)
 			(effects
 				(font
@@
 		)
 		(property "Datasheet" "https://www.nidec-components.com/e/catalog/switch/cas.pdf"
-			(at 60.96 180.34 0)
+			(at 55.88 180.34 0)
 			(effects
 				(font
@@
 		)
 		(property "Description" "Switch, single pole double throw"
-			(at 60.96 187.96 0)
+			(at 55.88 187.96 0)
 			(effects
 				(font
@@
 			)
 		)
-		(property "Value" "240Ω"
+		(property "Value" "1kΩ"
 			(at 232.41 81.788 90)
 			(effects
@@
 			)
 		)
-		(property "Value" "240Ω"
+		(property "Value" "1kΩ"
 			(at 232.41 100.838 90)
 			(effects
@@
 	(symbol
 		(lib_id "Device:Polyfuse")
-		(at 44.45 185.42 90)
+		(at 67.31 187.96 90)
 		(unit 1)
 		(exclude_from_sim no)
@@
 		(dnp no)
 		(property "Reference" "F1"
-			(at 44.45 179.07 90)
+			(at 67.31 181.61 90)
 			(effects
 				(font
@@
 		)
 		(property "Value" "MF-R050"
-			(at 44.45 181.61 90)
+			(at 67.31 184.15 90)
 			(effects
 				(font
@@
 		)
 		(property "Footprint" "00a:MF-R050"
-			(at 50.546 185.166 0)
+			(at 73.406 187.706 0)
 			(effects
 				(font
@@
 		)
 		(property "Datasheet" "~"
-			(at 44.45 185.42 0)
+			(at 67.31 187.96 0)
 			(effects
 				(font
@@
 		)
 		(property "Description" "Resettable fuse, polymeric positive temperature coefficient"
-			(at 44.45 185.42 0)
+			(at 67.31 187.96 0)
 			(effects
 				(font
